File: hardware_design/thermal_camera_v2.kicad_sch (KiCad schematic)
At the start: 52 parts, among them J1 Conn_01x04_Female, J2 Conn_01x01_Male, J3 Conn_01x07_Female, J4 Conn_01x01_Female, J5 USB_B_Mini, Q1 AP2312, Q2 AP2311, SW1 DTSMW69N, SW2 DTSMW69N, U1 STM32F205RCTx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

Commit message: Fix button part number, add components BOM
Parts:
- R1, R10, R3, R9: value 4k7 -> 3k3
- SW1, SW2: value DTSMW69N -> 1-1825910-4
- U1: value STM32F205RCTx -> STM32F205RC
- U2: value (none) -> LP2981-3.3; footprint (none) -> Package_TO_SOT_SMD:SOT-23-5
- U4: value M25PX32-VMW -> W25Q64
Changed lines of the file:
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@@
       (effects (font (size 1.27 1.27)) (justify left))
     )
-    (property "Value" "M25PX32-VMW" (id 1) (at 176.53 156.21 0)
+    (property "Value" "W25Q64" (id 1) (at 176.53 156.21 0)
       (effects (font (size 1.27 1.27)) (justify left))
     )
@@
     (in_bom yes) (on_board yes) (fields_autoplaced)
     (property "Reference" "U2" (id 0) (at 257.81 21.0652 0))
-    (property "Value" "" (id 1) (at 257.81 23.6021 0))
-    (property "Footprint" "" (id 2) (at 257.81 20.955 0)
+    (property "Value" "LP2981-3.3" (id 1) (at 257.81 23.6021 0))
+    (property "Footprint" "Package_TO_SOT_SMD:SOT-23-5" (id 2) (at 257.81 20.955 0)
       (effects (font (size 1.27 1.27)) hide)
     )
@@
       (effects (font (size 1.27 1.27)) (justify left))
     )
-    (property "Value" "DTSMW69N" (id 1) (at 177.673 34.7222 90)
+    (property "Value" "1-1825910-4" (id 1) (at 177.673 34.7222 90)
       (effects (font (size 1.27 1.27)) (justify left))
     )
@@
     (in_bom yes) (on_board yes) (fields_autoplaced)
     (property "Reference" "SW2" (id 0) (at 194.31 64.2325 0))
-    (property "Value" "DTSMW69N" (id 1) (at 194.31 67.0076 0))
+    (property "Value" "1-1825910-4" (id 1) (at 194.31 67.0076 0))
     (property "Footprint" "Button_Switch_THT:SW_PUSH_6mm" (id 2) (at 194.31 63.5 0)
       (effects (font (size 1.27 1.27)) hide)
@@
       (effects (font (size 1.27 1.27)) (justify right))
     )
-    (property "Value" "4k7" (id 1) (at 168.148 104.7366 0)
+    (property "Value" "3k3" (id 1) (at 168.148 104.7366 0)
       (effects (font (size 1.27 1.27)) (justify right))
     )
@@
       (effects (font (size 1.27 1.27)) (justify right))
     )
-    (property "Value" "4k7" (id 1) (at 175.768 104.7366 0)
+    (property "Value" "3k3" (id 1) (at 175.768 104.7366 0)
       (effects (font (size 1.27 1.27)) (justify right))
     )
@@
       (effects (font (size 1.27 1.27)) (justify right))
     )
-    (property "Value" "4k7" (id 1) (at 215.392 33.6166 0)
+    (property "Value" "3k3" (id 1) (at 215.392 33.6166 0)
       (effects (font (size 1.27 1.27)) (justify right))
     )
@@
       (effects (font (size 1.27 1.27)) (justify right))
     )
-    (property "Value" "4k7" (id 1) (at 202.438 53.9366 0)
+    (property "Value" "3k3" (id 1) (at 202.438 53.9366 0)
       (effects (font (size 1.27 1.27)) (justify right))
     )
@@
       (effects (font (size 1.27 1.27)) (justify left))
     )
-    (property "Value" "STM32F205RCTx" (id 1) (at 92.1894 177.6446 0)
+    (property "Value" "STM32F205RC" (id 1) (at 92.1894 177.6446 0)
       (effects (font (size 1.27 1.27)) (justify left))
     )
@@
     )
     (path "/ed6cd72f-4985-4265-a8c6-e1402f632187"
-      (reference "R1") (unit 1) (value "4k7") (footprint "Resistor_SMD:R_0603_1608Metric_Pad0.98x0.95mm_HandSolder")
+      (reference "R1") (unit 1) (value "3k3") (footprint "Resistor_SMD:R_0603_1608Metric_Pad0.98x0.95mm_HandSolder")
     )
     (path "/c497ce32-ebb0-414e-8505-ead96089a3d9"
@@
     )
     (path "/d0c2b49f-5c84-4339-a102-0bc70aca51aa"
-      (reference "R3") (unit 1) (value "4k7") (footprint "Resistor_SMD:R_0603_1608Metric_Pad0.98x0.95mm_HandSolder")
+      (reference "R3") (unit 1) (value "3k3") (footprint "Resistor_SMD:R_0603_1608Metric_Pad0.98x0.95mm_HandSolder")
     )
     (path "/c3629968-32ce-4033-b43b-b55c9505e176"
@@
     )
     (path "/989e2a84-b739-4f11-b473-447caf869367"
-      (reference "R9") (unit 1) (value "4k7") (footprint "Resistor_SMD:R_0603_1608Metric_Pad0.98x0.95mm_HandSolder")
+      (reference "R9") (unit 1) (value "3k3") (footprint "Resistor_SMD:R_0603_1608Metric_Pad0.98x0.95mm_HandSolder")
     )
     (path "/cbae8d6e-d8c7-4055-bdd8-8e2a628e2e20"
-      (reference "R10") (unit 1) (value "4k7") (footprint "Resistor_SMD:R_0603_1608Metric_Pad0.98x0.95mm_HandSolder")
+      (reference "R10") (unit 1) (value "3k3") (footprint "Resistor_SMD:R_0603_1608Metric_Pad0.98x0.95mm_HandSolder")
     )
     (path "/6edb0204-8483-434b-bb75-39a68473dbd2"
@@
     )
     (path "/38ed3450-4636-4ee0-a388-290538d99ea7"
-      (reference "SW1") (unit 1) (value "DTSMW69N") (footprint "Button_Switch_THT:SW_PUSH_6mm")
+      (reference "SW1") (unit 1) (value "1-1825910-4") (footprint "Button_Switch_THT:SW_PUSH_6mm")
     )
     (path "/7cb3cd96-5468-4447-a72a-1d69ce988849"
-      (reference "SW2") (unit 1) (value "DTSMW69N") (footprint "Button_Switch_THT:SW_PUSH_6mm")
+      (reference "SW2") (unit 1) (value "1-1825910-4") (footprint "Button_Switch_THT:SW_PUSH_6mm")
     )
     (path "/f73b5500-6337-4860-a114-6e307f65ec9f"
-      (reference "U1") (unit 1) (value "STM32F205RCTx") (footprint "Package_QFP:LQFP-64_10x10mm_P0.5mm")
+      (reference "U1") (unit 1) (value "STM32F205RC") (footprint "Package_QFP:LQFP-64_10x10mm_P0.5mm")
     )
     (path "/2ddfd9c2-a794-4ad9-be67-ca54dcea94fe"
@@
     )
     (path "/27260fd1-7e11-444d-9206-9db48718c252"
-      (reference "U4") (unit 1) (value "M25PX32-VMW") (footprint "Package_SO:SOIC-8W_5.3x5.3mm_P1.27mm")
+      (reference "U4") (unit 1) (value "W25Q64") (footprint "Package_SO:SOIC-8W_5.3x5.3mm_P1.27mm")
     )
     (path "/5767c56e-36f6-4ba4-83f2-6449f011099d"

Commit message: Switched XTAL footprint
Parts:
- removed Y1: 8MHz, TFT_footprints:XTAL_5030_china_unknown, symbol Device:Crystal_GND23
- added Y1: 8MHz, Crystal:Crystal_SMD_5032-4Pin_5.0x3.2mm, symbol Device:Crystal_GND24
Connections:
- net GND: now also Y1.4
- net at C13.1, U1.5 (PH0): now also Y1.1
- net at C12.1, U1.6 (PH1): now also Y1.3
